Commit message: xacro robot_wheel origin feature modified

File: src/ms_robot_description/urdf/robot_core.xacro (robot description, xacro)
@@ -13,9 +13,10 @@
         <parent link="base_link"/>
         <child link="left_wheel"/>
-        <origin xyz="0 0 0" rpy="0 0 0"/>
+        <origin xyz="0 ${wheel_separation/2} 0" rpy="0 0 0"/>
         <axis xyz="0 1 0"/>
     </joint>
     <link name="left_wheel">
         <visual>
+            <origin xyz="0 0 0" rpy="0 0 ${pi/2}"/>
             <geometry>
                 <mesh filename="package://ms_robot_description/meshes/visual/wheel.dae" scale="1 1 1"/>
@@ -26,9 +27,10 @@
         <parent link="base_link"/>
         <child link="right_wheel"/>
-        <origin xyz="0 0 0" rpy="0 0 0"/>
+        <origin xyz="0 ${-wheel_separation/2} 0" rpy="0 0 0"/>
         <axis xyz="0 1 0"/>
     </joint>
     <link name="right_wheel">
         <visual>
+            <origin xyz="0 0 0" rpy="0 0 ${-pi/2}"/>
             <geometry>
                 <mesh filename="package://ms_robot_description/meshes/visual/wheel.dae" scale="1 1 1"/>

Commit message: urdf modified

File: src/ms_robot_description/urdf/robot_core.xacro (robot description, xacro)
@@ -38,3 +38,41 @@
         </visual>
     </link>
+    <link name="ul_sensor_mount">
+        <visual>
+            <origin xyz="0 0 0" rpy="0 0 0"/>
+            <geometry>
+                <mesh filename="package://ms_robot_description/meshes/visual/ul_sensor.dae" scale="1 1 1"/>
+            </geometry>
+        </visual>
+    </link>
+    <joint name="ul_sensor_mount_fixed_joint" type="fixed">
+        <parent link="base_link"/>
+        <child link="ul_sensor_mount"/>
+        <origin xyz="0.03 0 0.01" rpy="0 0 0"/>
+    </joint>
+    <link name="ul_sensor_link"/>
+    <joint name="ul_sensor_link_fixed_joint" type="fixed">
+        <parent link="ul_sensor_mount"/>
+        <chile link="ul_sensor_link"/>
+        <origin xyz="0.02 0 0" rpy="0 0 0"/>
+    </joint>
+    <link name="ydlidar_lidar_mount">
+        <visual>
+            <origin xyz="0 0 0" rpy="0 0 0"/>
+            <geometry>
+                <mesh filename="package://ms_robot_description/meshes/visual/ydlidar_x2_assy.dae" scale="1 1 1"/>
+            </geometry>
+        </visual>
+    </link>
+    <joint name="lidar_mount_fixed_joint" type="fixed">
+        <parent link="base_link"/>
+        <child link="ydlidar_lidar_mount"/>
+        <origin xyz="-0.01 0 0.085" rpy="0 0 0"/>
+    </joint>
+    <link name="laser_link"/>
+    <joint name="laser_link_fixed_joint" type="fixed">
+        <parent link="ydlidar_lidar_mount"/>
+        <child link="laser_link"/>
+        <origin xyz="0 0 0.0425" rpy="0 0 0"/>
+    </joint>
 </robot>

Commit message: gazebo added

File: src/ms_robot_description/urdf/robot_core.xacro (robot description, xacro)
@@ -2,4 +2,11 @@
 <robot name="ms_robot" xmlns:xacro="http://www.ros.org/wiki/xacro">
     <xacro:property name="wheel_separation" value="0.180"/>
+    <xacro:property name="wheel_diameter" value="0.068"/>
+    <link name="base_footprint"/>
+    <joint name="base_link_fixed_joint" type="fixed">
+        <parent link="base_footprint"/>
+        <child link="base_link"/>
+        <origin xyz="0 0 ${wheel_diameter/2}" rpy="0 0 0"/>
+    </joint>
     <link name = "base_link">
         <visual>
@@ -9,4 +16,15 @@
             </geometry>
         </visual>
+        <collision>
+            <origin xyz="0 0 0" rpy="0 0 0"/>
+            <geometry>
+                <mesh filename="package://ms_robot_description/meshes/collision/base_link.stl" scale="1 1 1"/>
+            </geometry>
+        </collision>
+        <inertial>
+            <origin xyz="-0.02 0 0.028" rpy="0 0 0"/>
+            <mass value="2.0"/>
+            <inertia ixx="0.01" ixy="0" ixz="0" iyy="0.01" iyz="0" izz="0.01"/>
+        </inertial>
     </link>
     <joint name="left_wheel_joint" type="continuous">
@@ -23,9 +41,20 @@
             </geometry>
         </visual>
+        <collision>
+            <origin xyz="0 0 0" rpy="0 0 ${pi/2}"/>
+            <geometry>
+                <mesh filename="package://ms_robot_description/meshes/collision/wheel.stl" scale="1 1 1"/>
+            </geometry>
+        </collision>
+        <inertial>
+            <origin xyz="0 0 0" rpy="0 0 0"/>
+            <mass value="0.200"/>
+            <inertia ixx="0.1" ixy="0" ixz="0" iyy="0.1" iyz="0" izz="0.1"/>
+        </inertial>
     </link>
     <joint name="right_wheel_joint" type="continuous">
         <parent link="base_link"/>
         <child link="right_wheel"/>
-        <origin xyz="0 ${-wheel_separation/2} 0" rpy="0 0 0"/>
+        <origin xyz="0 ${-1 * wheel_separation/2} 0" rpy="0 0 0"/>
         <axis xyz="0 1 0"/>
     </joint>
@@ -37,4 +66,15 @@
             </geometry>
         </visual>
+        <collision>
+        <origin xyz="0 0 0" rpy="0 0 ${-1 * pi/2}"/>
+            <geometry>
+                <mesh filename="package://ms_robot_description/meshes/collision/wheel.stl" scale="1 1 1"/>
+            </geometry>
+        </collision>
+        <inertial>
+            <origin xyz="0 0 0" rpy="0 0 0"/>
+            <mass value="0.200"/>
+            <inertia ixx="0.1" ixy="0" ixz="0" iyy="0.1" iyz="0" izz="0.1"/>
+        </inertial>
     </link>
     <link name="ul_sensor_mount">
@@ -45,4 +85,15 @@
             </geometry>
         </visual>
+        <collision>
+            <origin xyz="0 0 0" rpy="0 0 0"/>
+            <geometry>
+                <mesh filename="package://ms_robot_description/meshes/collision/ul_sensor.stl" scale="1 1 1"/>
+            </geometry>
+        </collision>
+        <inertial>
+            <origin xyz="0.005 0 0.013" rpy="0 0 0"/>
+            <mass value="0.050000"/>
+            <inertia ixx="0.000005" ixy="0" ixz="-0.000001" iyy="0.000004" iyz="0" izz="0.000003"/>
+        </inertial>
     </link>
     <joint name="ul_sensor_mount_fixed_joint" type="fixed">
@@ -54,5 +105,5 @@
     <joint name="ul_sensor_link_fixed_joint" type="fixed">
         <parent link="ul_sensor_mount"/>
-        <chile link="ul_sensor_link"/>
+        <child link="ul_sensor_link"/>
         <origin xyz="0.02 0 0" rpy="0 0 0"/>
     </joint>
@@ -64,4 +115,15 @@
             </geometry>
         </visual>
+        <collision>
+        <origin xyz="0 0 0" rpy="0 0 0"/>
+            <geometry>
+                <mesh filename="package://ms_robot_description/meshes/collision/ydlidar_x2_assy.stl" scale="1 1 1"/>
+            </geometry>
+        </collision>
+        <inertial>
+            <origin xyz="0.007 0 0.025" rpy="0 0 0"/>
+            <mass value="0.150"/>
+            <inertia ixx="0.000058" ixy="0" ixz="0.000005" iyy="0.000099" iyz="0" izz="0.000103"/>
+        </inertial>
     </link>
     <joint name="lidar_mount_fixed_joint" type="fixed">
@@ -76,3 +138,33 @@
         <origin xyz="0 0 0.0425" rpy="0 0 0"/>
     </joint>
+    <link name="front_camera_mount">
+        <visual>
+            <origin xyz="0 0 0" rpy="0 0 0"/>
+            <geometry>
+                <mesh filename="package://ms_robot_description/meshes/visual/front_camera.dae" scale="1 1 1"/>
+            </geometry>
+        </visual>
+        <collision>
+            <origin xyz="0 0 0" rpy="0 0 0"/>
+            <geometry>
+            <mesh filename="package://ms_robot_description/meshes/collision/front_camera.stl" scale="1 1 1"/>
+            </geometry>
+        </collision>
+        <inertial>
+            <origin xyz="0.005 0 0.013" rpy="0 0 0"/>
+            <mass value="0.050000"/>
+            <inertia ixx="0.000005" ixy="0" ixz="-0.000001" iyy="0.000004" iyz="0" izz="0.000003"/>
+        </inertial>
+    </link>
+    <joint name="front_camera_mount_fixed_joint" type="fixed">
+        <parent link="base_link"/>
+        <child link="front_camera_mount"/>
+        <origin xyz="0.045 0 0.085" rpy="0 0 0"/>
+    </joint>
+    <link name="camera_link"/>
+    <joint name="camera_link_fixed_joint" type="fixed">
+        <parent link="front_camera_mount"/>
+        <child link="camera_link"/>
+        <origin xyz="0.0111 0 0.0193" rpy="0 ${pi/2} 0"/>
+    </joint>
 </robot>
